File: PCB.brd (EAGLE design)
At the start: 160 x 100 mm, 25 parts

Commit message: Add files via upload
Other:
- board size 160 x 100 mm -> 71.1 x 56.8 mm
Changed lines of the file:
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@@
 <board>
 <plain>
-<wire x1="0" y1="0" x2="160" y2="0" width="0" layer="20"/>
-<wire x1="160" y1="0" x2="160" y2="100" width="0" layer="20"/>
-<wire x1="160" y1="100" x2="0" y2="100" width="0" layer="20"/>
-<wire x1="0" y1="100" x2="0" y2="0" width="0" layer="20"/>
+<wire x1="7.62" y1="39.37" x2="78.72" y2="39.37" width="0" layer="20"/>
+<wire x1="78.72" y1="39.37" x2="78.72" y2="96.19" width="0" layer="20"/>
+<wire x1="78.72" y1="96.19" x2="7.62" y2="96.19" width="0" layer="20"/>
+<wire x1="7.62" y1="96.19" x2="7.62" y2="39.37" width="0" layer="20"/>
 <text x="24.13" y="48.26" size="1.778" layer="1">EMG Circuit
 Rev 1.0
@@
 </element>
 <element name="U$6" logical_identifier="U$6" library="adafruit" library_urn="urn:adsk.wipprod:fs.file:vf.Kp_dagt0Qs62-CKkMOB2yg" package="FIDUCIAL_1MM" package3d_urn="urn:adsk.eagle:package:6240632/1" value="FIDUCIAL" x="12.7" y="87.63" smashed="yes">
+<attribute name="MANUFACTURER" value="Bourns Inc." x="12.7" y="87.63" size="1.778" layer="27" display="off"/>
 </element>
 <element name="U$7" logical_identifier="U$7" library="adafruit" library_urn="urn:adsk.wipprod:fs.file:vf.Kp_dagt0Qs62-CKkMOB2yg" package="FIDUCIAL_1MM" package3d_urn="urn:adsk.eagle:package:6240632/1" value="FIDUCIAL" x="66.04" y="87.63" smashed="yes">
+<attribute name="MANUFACTURER" value="Bourns Inc." x="66.04" y="87.63" size="1.778" layer="27" display="off"/>
 </element>
 <element name="U$9" logical_identifier="U$9" library="adafruit" library_urn="urn:adsk.wipprod:fs.file:vf.Kp_dagt0Qs62-CKkMOB2yg" package="FIDUCIAL_1MM" package3d_urn="urn:adsk.eagle:package:6240632/1" value="FIDUCIAL" x="13.97" y="43.18" smashed="yes">
+<attribute name="MANUFACTURER" value="Bourns Inc." x="13.97" y="43.18" size="1.778" layer="27" display="off"/>
 </element>
 <element name="R14" logical_identifier="R14" library="Tutorial - Fusion 360" library_urn="urn:adsk.eagle:library:16997205" package="RESC1005X40" package3d_urn="urn:adsk.eagle:package:16378568/5" value="1 MΩ" x="53.34" y="59.69" smashed="yes">
@@
 <contactref element="R5" pad="2"/>
 <contactref element="R4" pad="2"/>
-<wire x1="34.23555" y1="78.2325" x2="34.29" y2="78.2325" width="0.1524" layer="1"/>
-<wire x1="33.72805" y1="78.74" x2="34.23555" y2="78.2325" width="0.254" layer="1"/>
-<wire x1="31.12" y1="78.74" x2="33.72805" y2="78.74" width="0.254" layer="1"/>
+<wire x1="34.29" y1="78.2325" x2="34.23555" y2="78.2325" width="0.1524" layer="1"/>
+<wire x1="34.23555" y1="78.2325" x2="33.72805" y2="78.74" width="0.254" layer="1"/>
+<wire x1="33.72805" y1="78.74" x2="31.12" y2="78.74" width="0.254" layer="1"/>
 <wire x1="31.12" y1="78.74" x2="31.12" y2="81.28" width="0.254" layer="1"/>
 <wire x1="31.12" y1="78.74" x2="31.12" y2="75.79" width="0.254" layer="1"/>
@@
 <wire x1="39.37" y1="76.9854" x2="38.9602" y2="77.3952" width="0.254" layer="1"/>
 <wire x1="38.9602" y1="77.3952" x2="38.93971875" y2="77.3952" width="0.254" layer="1"/>
-<wire x1="34.29" y1="78.2325" x2="38.10241875" y2="78.2325" width="0.254" layer="1"/>
+<wire x1="38.10241875" y1="78.2325" x2="34.29" y2="78.2325" width="0.254" layer="1"/>
 <wire x1="38.93971875" y1="77.3952" x2="38.10241875" y2="78.2325" width="0.254" layer="1"/>
 </signal>
@@
 <wire x1="36.83" y1="83.3125" x2="36.83" y2="81.28" width="0.381" layer="1"/>
 <wire x1="20.95" y1="78.74" x2="22.22" y2="78.74" width="0.381" layer="1"/>
-<wire x1="20.95" y1="78.74" x2="20.32" y2="78.11" width="0.381" layer="1"/>
-<wire x1="20.32" y1="78.11" x2="20.32" y2="77.47" width="0.381" layer="1"/>
+<wire x1="20.32" y1="78.11" x2="20.95" y2="78.74" width="0.381" layer="1"/>
+<wire x1="20.32" y1="77.47" x2="20.32" y2="78.11" width="0.381" layer="1"/>
 <via x="28.5524" y="69.85" extent="1-16" drill="0.35" alwaysstop="yes">
 </via>
@@
 <via x="44.45" y="87.63" extent="1-16" drill="0.35" alwaysstop="yes">
 </via>
-<wire x1="45.08" y1="85.4876" x2="44.66" y2="85.4876" width="0.1524" layer="1"/>
-<wire x1="44.66" y1="85.4876" x2="44.45" y2="85.6976" width="0.1524" layer="1"/>
-<wire x1="44.45" y1="85.6976" x2="44.45" y2="87.63" width="0.254" layer="1"/>
+<wire x1="44.66" y1="85.4876" x2="45.08" y2="85.4876" width="0.1524" layer="1"/>
+<wire x1="44.45" y1="85.6976" x2="44.66" y2="85.4876" width="0.1524" layer="1"/>
+<wire x1="44.45" y1="87.63" x2="44.45" y2="85.6976" width="0.254" layer="1"/>
 <wire x1="44.45" y1="87.63" x2="55.88" y2="87.63" width="0.254" layer="16"/>
 <wire x1="55.88" y1="87.63" x2="55.88" y2="80.01" width="0.254" layer="16"/>
@@
 </via>
 <wire x1="60.32" y1="85.09" x2="58.42" y2="85.09" width="0.254" layer="1"/>
-<wire x1="60.96" y1="55.88" x2="60.96" y2="76.2" width="0.254" layer="16"/>
+<wire x1="60.96" y1="76.2" x2="60.96" y2="55.88" width="0.254" layer="16"/>
 <wire x1="60.96" y1="76.2" x2="58.42" y2="78.74" width="0.254" layer="16"/>
 <wire x1="58.42" y1="85.09" x2="58.42" y2="78.74" width="0.254" layer="16"/>
@@
 <contactref element="B1" pad="A1"/>
 <contactref element="R13" pad="2"/>
-<wire x1="63.59848125" y1="57.67151875" x2="62.04108125" y2="56.11411875" width="0.254" layer="16"/>
+<wire x1="62.04108125" y1="56.11411875" x2="63.59848125" y2="57.67151875" width="0.254" layer="16"/>
 <wire x1="62.04108125" y1="56.11411875" x2="62.04108125" y2="44.2889125" width="0.254" layer="16"/>
 <wire x1="62.04108125" y1="44.2889125" x2="62.30759375" y2="44.0224" width="0.254" layer="16"/>
